Commit message: 🔧  Modified joint order to make it mujoco compatible

File: urdf/rg2_macro.xacro (robot description, xacro)
@@ -22,6 +22,20 @@
       <mimic joint="${prefix}finger_joint" multiplier="1" offset="0" />
     </joint>
+    <link name="${prefix}${fingerprefix}_finger_tip" />
+    <joint name="${prefix}${fingerprefix}_finger_tip_joint" type="fixed">
+      <origin xyz="0 0.019 0.038" rpy="0 0 0" />
+      <parent link="${prefix}${fingerprefix}_inner_finger" />
+      <child link="${prefix}${fingerprefix}_finger_tip" />
+    </joint>
   </xacro:macro>
   <xacro:macro name="finger_joint" params="prefix">
+    <link name="${prefix}finger_width_mock_link"/>
+    <joint name="${prefix}finger_width" type="prismatic">
+      <origin xyz="0 0 0" rpy="0 0 0" />
+      <parent link="${prefix}onrobot_base_link" />
+      <child link="${prefix}finger_width_mock_link" />
+      <axis xyz="0 0 1" />
+      <limit lower="0" upper="0.110" velocity="0.127" effort="40" />
+    </joint>
     <joint name="${prefix}finger_joint" type="revolute">
       <origin xyz="0 -0.017178 0.125797" rpy="0 0 0" />
@@ -45,26 +59,10 @@
     <xacro:finger_joints prefix="${prefix}" fingerprefix="right" reflect="-1.0"/>
   </xacro:macro>
-  <xacro:macro name="finger_tips" params="prefix">
-    <link name="${prefix}left_finger_tip"/>
-    <link name="${prefix}right_finger_tip"/>
-    <link name="${prefix}gripper_tcp"/>
-    <joint name="${prefix}left_finger_tip_joint" type="fixed">
-      <origin xyz="0 0.019 0.038" rpy="0 0 0" />
-      <parent link="${prefix}left_inner_finger" />
-      <child link="${prefix}left_finger_tip" />
-    </joint>
-    <joint name="${prefix}finger_width" type="prismatic">
-      <origin xyz="0 0 0" rpy="${pi} 0 0" />
-      <parent link="${prefix}left_finger_tip" />
-      <child link="${prefix}right_finger_tip" />
-      <axis xyz="0 -1 0" />
-      <limit lower="0" upper="0.110" velocity="0.127" effort="40" />
-    </joint>
-    <joint name="${prefix}tcp_joint" type="fixed">
-      <origin xyz="0 0 0.218" rpy="0 0 0" />
-      <parent link="${prefix}onrobot_base_link" />
-      <child link="${prefix}gripper_tcp" />
-    </joint>
-  </xacro:macro>
+  <link name="${prefix}gripper_tcp" />
+  <joint name="${prefix}tcp_joint" type="fixed">
+    <origin xyz="0 0 0.218" rpy="0 0 0" />
+    <parent link="${prefix}onrobot_base_link" />
+    <child link="${prefix}gripper_tcp" />
+  </joint>
   <xacro:macro name="onrobot_rg2" params="prefix">
     <xacro:onrobot_base_link prefix="${prefix}" />
@@ -72,5 +70,4 @@
     <xacro:finger_links prefix="${prefix}" fingerprefix="right"/>
     <xacro:finger_joint prefix="${prefix}"/>
-    <xacro:finger_tips prefix="${prefix}"/>
     <xacro:right_outer_knuckle_joint prefix="${prefix}"/>
     <xacro:transmission_macro prefix="${prefix}" joint_name="finger_width"/>

File: urdf/rg6_macro.xacro (robot description, xacro)
@@ -22,6 +22,20 @@
       <mimic joint="${prefix}finger_joint" multiplier="1" offset="0" />
     </joint>
+    <link name="${prefix}${fingerprefix}_finger_tip"/>
+    <joint name="${prefix}${fingerprefix}_finger_tip_joint" type="fixed">
+      <origin xyz="0 0.025 0.052" rpy="0 0 0" />
+      <parent link="${prefix}${fingerprefix}_inner_finger" />
+      <child link="${prefix}${fingerprefix}_finger_tip" />
+    </joint>
   </xacro:macro>
   <xacro:macro name="finger_joint" params="prefix">
+    <link name="${prefix}finger_width_mock_link"/>
+    <joint name="${prefix}finger_width" type="prismatic">
+      <origin xyz="0 0 0" rpy="0 0 0" />
+      <parent link="${prefix}onrobot_base_link" />
+      <child link="${prefix}finger_width_mock_link" />
+      <axis xyz="0 0 1" />
+      <limit lower="0" upper="0.160" velocity="0.160" effort="120" />
+    </joint>
     <joint name="${prefix}finger_joint" type="revolute">
       <origin xyz="0 -0.024112 0.136813" rpy="0 0 0" />
@@ -45,26 +59,10 @@
     <xacro:finger_joints prefix="${prefix}" fingerprefix="right" reflect="-1.0"/>
   </xacro:macro>
-  <xacro:macro name="finger_tips" params="prefix">
-    <link name="${prefix}left_finger_tip"/>
-    <link name="${prefix}right_finger_tip"/>
-    <link name="${prefix}gripper_tcp"/>
-    <joint name="${prefix}left_finger_tip_joint" type="fixed">
-      <origin xyz="0 0.025 0.058" rpy="0 0 0" />
-      <parent link="${prefix}left_inner_finger" />
-      <child link="${prefix}left_finger_tip" />
-    </joint>
-    <joint name="${prefix}finger_width" type="prismatic">
-      <origin xyz="0 0 0" rpy="${pi} 0 0" />
-      <parent link="${prefix}left_finger_tip" />
-      <child link="${prefix}right_finger_tip" />
-      <axis xyz="0 -1 0" />
-      <limit lower="0" upper="0.160" velocity="0.160" effort="120" />
-    </joint>
-    <joint name="${prefix}tcp_joint" type="fixed">
-      <origin xyz="0 0 0.268" rpy="0 0 0" />
-      <parent link="${prefix}onrobot_base_link" />
-      <child link="${prefix}gripper_tcp" />
-    </joint>
-  </xacro:macro>
+  <link name="${prefix}gripper_tcp"/>
+  <joint name="${prefix}tcp_joint" type="fixed">
+    <origin xyz="0 0 0.268" rpy="0 0 0" />
+    <parent link="${prefix}onrobot_base_link" />
+    <child link="${prefix}gripper_tcp" />
+  </joint>
   <xacro:macro name="onrobot_rg6" params="prefix">
     <xacro:onrobot_base_link prefix="${prefix}" />
@@ -72,5 +70,4 @@
     <xacro:finger_links prefix="${prefix}" fingerprefix="right"/>
     <xacro:finger_joint prefix="${prefix}"/>
-    <xacro:finger_tips prefix="${prefix}"/>
     <xacro:right_outer_knuckle_joint prefix="${prefix}"/>
     <xacro:transmission_macro prefix="${prefix}" joint_name="finger_width"/>
