Commit message: 🔧 Added ROS2 Control tags

File: urdf/onrobot.urdf.xacro (robot description, xacro)
@@ -6,8 +6,10 @@
     <xacro:arg name="name" default="onrobot"/>
     <xacro:arg name="sim_gazebo" default="false"/>
+    <xacro:arg name="use_fake_hardware" default="false"/>
     <!-- Import the OnRobot macro -->
     <xacro:include filename="$(find onrobot_description)/urdf/onrobot_macro.xacro"/>
     <!-- Create OnRobot instance -->
-    <xacro:onrobot onrobot_type="$(arg onrobot_type)" prefix="$(arg prefix)"/>
+    <xacro:onrobot onrobot_type="$(arg onrobot_type)" prefix="$(arg prefix)"
+        sim_gazebo="$(arg sim_gazebo)" use_fake_hardware="$(arg use_fake_hardware)"/>
     <!-- Create link fixed to the world -->
     <link name="world" />
@@ -17,7 +19,3 @@
         <child link="$(arg prefix)onrobot_base_link"/>
     </joint>
-    <!-- Optional Gazebo plugin if simulation is enabled -->
-    <xacro:if value="$(arg sim_gazebo)">
-        <xacro:gazebo_plugin prefix="$(arg prefix)"/>
-    </xacro:if>
 </robot>

File: urdf/onrobot_macro.xacro (robot description, xacro)
@@ -2,5 +2,5 @@
 <robot xmlns:xacro="http://wiki.ros.org/xacro">
     <!-- Include the macro file for the specific OnRobot model -->
-    <xacro:macro name="onrobot" params="onrobot_type prefix">
+    <xacro:macro name="onrobot" params="onrobot_type prefix sim_gazebo use_fake_hardware">
         <xacro:property name="onrobot_type" value="$(arg onrobot_type)"/>
         <xacro:if value="${onrobot_type == 'rg2'}">
@@ -12,4 +12,29 @@
             <xacro:onrobot_rg6 prefix="${prefix}"/>
         </xacro:if>
+        <!-- Enable the gazebo plugin for simulation -->
+        <xacro:if value="$(arg sim_gazebo)">
+            <gazebo>
+                <plugin filename="libgazebo_ros2_control.so" name="gazebo_ros2_control"/>
+            </gazebo>
+        </xacro:if>
+        <!-- Define the OnRobot gripper hardware interface for ROS 2 control -->
+        <ros2_control name="OnRobotGripper" type="actuator">
+            <hardware>
+                <xacro:if value="${sim_gazebo}">
+                    <plugin>gazebo_ros2_control/GazeboSystem</plugin>
+                </xacro:if>
+                <xacro:if value="${use_fake_hardware}">
+                    <plugin>mock_components/GenericSystem</plugin>
+                    <param name="calculate_dynamics">false</param>
+                </xacro:if>
+                <xacro:unless value="${sim_gazebo}">
+                    <plugin>onrobot_driver/RGHardwareInterface</plugin>
+                </xacro:unless>
+            </hardware>
+            <joint name="finger_width">
+                <command_interface name="position"/>
+                <state_interface name="position"/>
+            </joint>
+        </ros2_control>
     </xacro:macro>
 </robot>

Commit message: 🔧 Configurable connection types for ROS 2 control

File: urdf/onrobot.urdf.xacro (robot description, xacro)
@@ -7,9 +7,21 @@
     <xacro:arg name="sim_gazebo" default="false"/>
     <xacro:arg name="use_fake_hardware" default="false"/>
+    <xacro:arg name="connection_type" default="serial"/>
+    <xacro:arg name="device" default="/tmp/ttyUR"/>
+    <xacro:arg name="ip_address" default="192.168.1.1"/>
+    <xacro:arg name="port" default="502"/>
     <!-- Import the OnRobot macro -->
     <xacro:include filename="$(find onrobot_description)/urdf/onrobot_macro.xacro"/>
     <!-- Create OnRobot instance -->
-    <xacro:onrobot onrobot_type="$(arg onrobot_type)" prefix="$(arg prefix)"
-        sim_gazebo="$(arg sim_gazebo)" use_fake_hardware="$(arg use_fake_hardware)"/>
+    <xacro:onrobot
+        onrobot_type="$(arg onrobot_type)"
+        prefix="$(arg prefix)"
+        sim_gazebo="$(arg sim_gazebo)"
+        use_fake_hardware="$(arg use_fake_hardware)"
+        connection_type="$(arg connection_type)"
+        device="$(arg device)"
+        ip_address="$(arg ip_address)"
+        port="$(arg port)"
+    />
     <!-- Create link fixed to the world -->
     <link name="world" />

File: urdf/onrobot_macro.xacro (robot description, xacro)
@@ -2,5 +2,15 @@
 <robot xmlns:xacro="http://wiki.ros.org/xacro">
     <!-- Include the macro file for the specific OnRobot model -->
-    <xacro:macro name="onrobot" params="onrobot_type prefix sim_gazebo use_fake_hardware">
+    <xacro:macro name="onrobot"
+        params="
+        onrobot_type
+        prefix:=''
+        sim_gazebo:=false
+        use_fake_hardware:=false
+        connection_type:=serial
+        device:=/tmp/ttyUR
+        ip_address:=192.168.1.1
+        port:=502
+        ">
         <xacro:property name="onrobot_type" value="$(arg onrobot_type)"/>
         <xacro:if value="${onrobot_type == 'rg2'}">
@@ -28,9 +38,15 @@
                     <param name="calculate_dynamics">false</param>
                 </xacro:if>
-                <xacro:unless value="${sim_gazebo}">
+                <xacro:unless value="${sim_gazebo or use_fake_hardware}">
                     <plugin>onrobot_driver/RGHardwareInterface</plugin>
+                    <param name="onrobot_type">${onrobot_type}</param>
+                    <param name="prefix">${prefix}</param>
+                    <param name="connection_type">${connection_type}</param>
+                    <param name="device">${device}</param>
+                    <param name="ip_address">${ip_address}</param>
+                    <param name="port">${port}</param>
                 </xacro:unless>
             </hardware>
-            <joint name="finger_width">
+            <joint name="${prefix}finger_width">
                 <command_interface name="position"/>
                 <state_interface name="position"/>
