Commit message: 🔧  Unified onrobot xacros for better modularity

File: urdf/inc/rg_common.xacro (robot description, xacro)
@@ -3,7 +3,7 @@
   <!-- Define RG type -->
   <xacro:arg name="type" default="rg2" />
-  <xacro:property name="onrobot_type" value="$(arg type)" />
+  <xacro:property name="type" value="$(arg type)" />
   <xacro:macro name="onrobot_base_link" params="prefix">
-    <xacro:if value="${onrobot_type == 'rg2'}">
+    <xacro:if value="${type == 'rg2'}">
       <xacro:property name="mass" value="0.78" />
       <xacro:property name="ixx" value="1.0E-03" />
@@ -14,5 +14,5 @@
       <xacro:property name="izz" value="1.0E-03" />
     </xacro:if>
-    <xacro:if value="${onrobot_type == 'rg6'}">
+    <xacro:if value="${type == 'rg6'}">
       <xacro:property name="mass" value="1.25" />
       <xacro:property name="ixx" value="1.0E-03" />
@@ -32,5 +32,5 @@
         <origin xyz="0 0 0" rpy="0 0 0" />
         <geometry>
-          <mesh filename="package://onrobot_description/meshes/${onrobot_type}/visual/base_link.stl" />
+          <mesh filename="package://onrobot_description/meshes/${type}/visual/base_link.stl" />
         </geometry>
         <material name="">
@@ -41,5 +41,5 @@
         <origin xyz="0 0 0" rpy="0 0 0" />
         <geometry>
-          <mesh filename="package://onrobot_description/meshes/${onrobot_type}/collision/base_link.stl" />
+          <mesh filename="package://onrobot_description/meshes/${type}/collision/base_link.stl" />
         </geometry>
       </collision>
@@ -62,5 +62,5 @@
         <origin xyz="0 0 0" rpy="0 0 0" />
         <geometry>
-          <mesh filename="package://onrobot_description/meshes/${onrobot_type}/visual/outer_knuckle.stl" />
+          <mesh filename="package://onrobot_description/meshes/${type}/visual/outer_knuckle.stl" />
         </geometry>
         <material name="">
@@ -71,5 +71,5 @@
         <origin xyz="0 0 0" rpy="0 0 0" />
         <geometry>
-          <mesh filename="package://onrobot_description/meshes/${onrobot_type}/collision/outer_knuckle.stl" />
+          <mesh filename="package://onrobot_description/meshes/${type}/collision/outer_knuckle.stl" />
         </geometry>
       </collision>
@@ -92,5 +92,5 @@
         <origin xyz="0 0 0" rpy="0 0 0" />
         <geometry>
-          <mesh filename="package://onrobot_description/meshes/${onrobot_type}/visual/inner_knuckle.stl" />
+          <mesh filename="package://onrobot_description/meshes/${type}/visual/inner_knuckle.stl" />
         </geometry>
         <material name="">
@@ -101,5 +101,5 @@
         <origin xyz="0 0 0" rpy="0 0 0" />
         <geometry>
-          <mesh filename="package://onrobot_description/meshes/${onrobot_type}/collision/inner_knuckle.stl" />
+          <mesh filename="package://onrobot_description/meshes/${type}/collision/inner_knuckle.stl" />
         </geometry>
       </collision>
@@ -122,5 +122,5 @@
         <origin xyz="0 0 0" rpy="0 0 0" />
         <geometry>
-          <mesh filename="package://onrobot_description/meshes/${onrobot_type}/visual/inner_finger.stl" />
+          <mesh filename="package://onrobot_description/meshes/${type}/visual/inner_finger.stl" />
         </geometry>
         <material name="">
@@ -131,5 +131,5 @@
         <origin xyz="0 0 0" rpy="0 0 0" />
         <geometry>
-          <mesh filename="package://onrobot_description/meshes/${onrobot_type}/collision/inner_finger.stl" />
+          <mesh filename="package://onrobot_description/meshes/${type}/collision/inner_finger.stl" />
         </geometry>
       </collision>

File: urdf/onrobot.urdf.xacro (robot description, xacro)
@@ -2,11 +2,12 @@
 <robot xmlns:xacro="http://wiki.ros.org/xacro" name="$(arg name)">
     <!-- Arguments -->
+    <xacro:arg name="onrobot_type" default="rg2"/>
+    <xacro:arg name="prefix" default=""/>
     <xacro:arg name="name" default="onrobot"/>
-    <xacro:arg name="prefix" default=""/>
     <xacro:arg name="sim_gazebo" default="false"/>
-    <!-- Import the RG2-specific macro file -->
-    <xacro:include filename="$(find onrobot_description)/urdf/rg2_macro.xacro"/>
-    <!-- Create RG2 instance -->
-    <xacro:onrobot_rg2 prefix="$(arg prefix)"/>
+    <!-- Import the OnRobot macro -->
+    <xacro:include filename="$(find onrobot_description)/urdf/onrobot_macro.xacro"/>
+    <!-- Create OnRobot instance -->
+    <xacro:onrobot onrobot_type="$(arg onrobot_type)" prefix="$(arg prefix)"/>
     <!-- Create link fixed to the world -->
     <link name="world" />

File: urdf/rg2_macro.xacro (robot description, xacro)
@@ -59,5 +59,5 @@
       <child link="${prefix}right_finger_tip" />
       <axis xyz="0 -1 0" />
-      <limit lower="0" upper="0.110" velocity="100.0" effort="1000" />
+      <limit lower="0" upper="0.110" velocity="0.127" effort="40" />
     </joint>
     <joint name="${prefix}tcp_joint" type="fixed">
@@ -67,5 +67,4 @@
     </joint>
   </xacro:macro>
-  <xacro:arg name="type" default="rg2" />
   <xacro:macro name="onrobot_rg2" params="prefix">
     <xacro:onrobot_base_link prefix="${prefix}" />

File: urdf/rg6_macro.xacro (robot description, xacro)
@@ -59,5 +59,5 @@
       <child link="${prefix}right_finger_tip" />
       <axis xyz="0 -1 0" />
-      <limit lower="0" upper="0.160" velocity="100.0" effort="1000" />
+      <limit lower="0" upper="0.160" velocity="0.160" effort="120" />
     </joint>
     <joint name="${prefix}tcp_joint" type="fixed">

Commit message: 🐛  Fixed "sim_gazebo" arg bug

File: urdf/inc/rg_common.xacro (robot description, xacro)
@@ -1,9 +1,6 @@
 <?xml version="1.0"?>
 <robot xmlns:xacro="http://www.ros.org/wiki/xacro">
-  <!-- Define RG type -->
-  <xacro:arg name="type" default="rg2" />
-  <xacro:property name="type" value="$(arg type)" />
   <xacro:macro name="onrobot_base_link" params="prefix">
-    <xacro:if value="${type == 'rg2'}">
+    <xacro:if value="${onrobot_type == 'rg2'}">
       <xacro:property name="mass" value="0.78" />
       <xacro:property name="ixx" value="1.0E-03" />
@@ -14,5 +11,5 @@
       <xacro:property name="izz" value="1.0E-03" />
     </xacro:if>
-    <xacro:if value="${type == 'rg6'}">
+    <xacro:if value="${onrobot_type == 'rg6'}">
       <xacro:property name="mass" value="1.25" />
       <xacro:property name="ixx" value="1.0E-03" />
@@ -32,5 +29,5 @@
         <origin xyz="0 0 0" rpy="0 0 0" />
         <geometry>
-          <mesh filename="package://onrobot_description/meshes/${type}/visual/base_link.stl" />
+          <mesh filename="package://onrobot_description/meshes/${onrobot_type}/visual/base_link.stl" />
         </geometry>
         <material name="">
@@ -41,5 +38,5 @@
         <origin xyz="0 0 0" rpy="0 0 0" />
         <geometry>
-          <mesh filename="package://onrobot_description/meshes/${type}/collision/base_link.stl" />
+          <mesh filename="package://onrobot_description/meshes/${onrobot_type}/collision/base_link.stl" />
         </geometry>
       </collision>
@@ -62,5 +59,5 @@
         <origin xyz="0 0 0" rpy="0 0 0" />
         <geometry>
-          <mesh filename="package://onrobot_description/meshes/${type}/visual/outer_knuckle.stl" />
+          <mesh filename="package://onrobot_description/meshes/${onrobot_type}/visual/outer_knuckle.stl" />
         </geometry>
         <material name="">
@@ -71,5 +68,5 @@
         <origin xyz="0 0 0" rpy="0 0 0" />
         <geometry>
-          <mesh filename="package://onrobot_description/meshes/${type}/collision/outer_knuckle.stl" />
+          <mesh filename="package://onrobot_description/meshes/${onrobot_type}/collision/outer_knuckle.stl" />
         </geometry>
       </collision>
@@ -92,5 +89,5 @@
         <origin xyz="0 0 0" rpy="0 0 0" />
         <geometry>
-          <mesh filename="package://onrobot_description/meshes/${type}/visual/inner_knuckle.stl" />
+          <mesh filename="package://onrobot_description/meshes/${onrobot_type}/visual/inner_knuckle.stl" />
         </geometry>
         <material name="">
@@ -101,5 +98,5 @@
         <origin xyz="0 0 0" rpy="0 0 0" />
         <geometry>
-          <mesh filename="package://onrobot_description/meshes/${type}/collision/inner_knuckle.stl" />
+          <mesh filename="package://onrobot_description/meshes/${onrobot_type}/collision/inner_knuckle.stl" />
         </geometry>
       </collision>
@@ -122,5 +119,5 @@
         <origin xyz="0 0 0" rpy="0 0 0" />
         <geometry>
-          <mesh filename="package://onrobot_description/meshes/${type}/visual/inner_finger.stl" />
+          <mesh filename="package://onrobot_description/meshes/${onrobot_type}/visual/inner_finger.stl" />
         </geometry>
         <material name="">
@@ -131,5 +128,5 @@
         <origin xyz="0 0 0" rpy="0 0 0" />
         <geometry>
-          <mesh filename="package://onrobot_description/meshes/${type}/collision/inner_finger.stl" />
+          <mesh filename="package://onrobot_description/meshes/${onrobot_type}/collision/inner_finger.stl" />
         </geometry>
       </collision>

File: urdf/onrobot_macro.xacro (robot description, xacro)
@@ -13,5 +13,4 @@
         port:=502
         ">
-        <xacro:property name="onrobot_type" value="$(arg onrobot_type)"/>
         <xacro:if value="${onrobot_type == 'rg2'}">
             <xacro:include filename="$(find onrobot_description)/urdf/rg2_macro.xacro"/>
@@ -23,5 +22,5 @@
         </xacro:if>
         <!-- Enable the gazebo plugin for simulation -->
-        <xacro:if value="$(arg sim_gazebo)">
+        <xacro:if value="${sim_gazebo}">
             <gazebo>
                 <plugin filename="libgazebo_ros2_control.so" name="gazebo_ros2_control"/>

File: urdf/rg2_macro.xacro (robot description, xacro)
@@ -1,5 +1,5 @@
 <?xml version="1.0"?>
 <robot xmlns:xacro="http://ros.org/wiki/xacro">
-  <xacro:arg name="type" default="rg2" />
+  <xacro:property name="onrobot_type" value="rg2" />
   <xacro:include filename="$(find onrobot_description)/urdf/inc/rg_common.xacro" />
   <xacro:macro name="inner_knuckle_joint" params="prefix fingerprefix reflect">

File: urdf/rg6_macro.xacro (robot description, xacro)
@@ -1,5 +1,5 @@
 <?xml version="1.0"?>
 <robot xmlns:xacro="http://ros.org/wiki/xacro">
-  <xacro:arg name="type" default="rg6" />
+  <xacro:property name="onrobot_type" value="rg6" />
   <xacro:include filename="$(find onrobot_description)/urdf/inc/rg_common.xacro" />
   <xacro:macro name="inner_knuckle_joint" params="prefix fingerprefix reflect">
